File: laser_diode_driver/laser_diode_driver.kicad_sch (KiCad schematic)
At the start: 13 parts, among them IC1 AL8843SP-13, IC2 LMH6642MA_NOPB, J1 12V IN, J2 0-5V Pangolin, J3 LASER OUT

Commit message: elo skonczone chyba
Parts:
- removed D1: 16V, symbol Device:D_Small
- removed R2: 11k, symbol Device:R_Small
- removed R3: 8.2k, symbol Device:R_Small
- added C2, C3: 100nF, Capacitor_SMD:C_1206_3216Metric_Pad1.33x1.80mm_HandSolder, symbol Device:C_Small
- added D2: 40V 3A, Diode_SMD:D_SMA_Handsoldering, symbol Device:D_Schottky_Small
- added IC3: MC33275ST-5.0T3G, SOT230P700X175-4N, symbol SamacSys_Parts:MC33275ST-5.0T3G
- L1: value ? -> 68uH 2A; footprint (none) -> SamacSys_Parts:INDPM172172X700N
- R1: value ? -> R052; footprint (none) -> Resistor_SMD:R_0201_0603Metric_Pad0.64x0.40mm_HandSolder
- R4, R5: footprint (none) -> Resistor_SMD:R_1206_3216Metric_Pad1.30x1.75mm_HandSolder
Connections:
- net +12V: now also C3.1, D2.1 (K), IC3.1 (VIN)
- net GND: now also C2.2, C3.2, IC3.2 (GND_1), IC3.4 (GND_2)
- net +5V: now reaches IC2.7 (V+)
- net +5V: now also C2.1, IC3.3 (VOUT)
- net at IC1.7 (SW_1), IC1.8 (SW_2), L1.1: now also D2.2 (A)
Other:
- moved on the sheet: C1, IC1, J2, J3, L1, R1, R4, R5

Commit message: initializing repo with existing schematics
Parts:
- removed J2: 0-5V Pangolin, TerminalBlock:TerminalBlock_bornier-2_P5.08mm, symbol Connector:Screw_Terminal_01x02
- added J2: Pango ILDA, symbol Connector:Screw_Terminal_01x03
- added R6: 1k, Resistor_SMD:R_1206_3216Metric_Pad1.30x1.75mm_HandSolder, symbol Device:R_Small
- R5: value 10k -> 500
Connections:
- net GND: now also J2.1 (Pin_1); no longer R5.2
- net at IC1.5 (CTRL), IC2.6 (OUTPUT): now also R5.2; no longer IC2.2 (-IN)
- net at R4.2, R5.1: now also IC2.2 (-IN); no longer IC2.3 (+IN)
- net Pango renamed Pango -
- net Pango -: now also J2.2 (Pin_2)
- new net: IC2.3 (+IN), R6.2
- new net Pango +: J2.3 (Pin_3), R6.1
Other:
- moved on the sheet: R4, R5
